Commit message: Add comments.

File: claw_example/claw_description/urdf/claw.urdf.xacro (robot description, xacro)
@@ -1,23 +1,50 @@
+<!--
+  urdf.xacro file extension indicates that this urdf file should not be directly used but included in another urdf file.
+  You will notice that this file isn't directly used anywhere within claw_example except claw.xacro. This file will make more sense when we want to combine it with another robot model.
+  This file contains the "description" i.e. links, joints, actuators, etc of our robot.
+ -->
 <?xml version="1.0" ?>
+<!-- The name of the robot is given here. xmlns:xacro is mandatory for xacro files. -->
 <robot name="claw" xmlns:xacro="http://ros.org/wiki/xacro">
+  <!--
+    This is the start of a macro block called "claw".
+    The macro block takes in 3 arguments:
+      - prefix is literally a prefix or "namespace within the string".
+      - parent is the name of the parent link of the claw.
+      - *origin is the tag for the origin.
+    * denotes that the variable is a tag. Literally <origin xyz=... />
+  -->
   <xacro:macro name="claw" params="prefix parent *origin">
+    <!-- This joint fixes the claw to an external parent link (could be the world or another robot). -->
     <joint name="${prefix}claw_flange" type="fixed">
       <parent link="${parent}"/>
       <child link="${prefix}base_link"/>
+      <!-- xacro:insert_block means place the tag here. Specify the positional relationship between parent and child links. -->
       <xacro:insert_block name="origin"/>
     </joint>
+    <!-- Define a link for mesh base_link.STL. -->
     <link name="${prefix}base_link">
+      <!-- Defines what the link looks like. -->
       <visual>
+        <!-- Shape of object. -->
         <geometry>
           <mesh filename="package://claw_description/meshes/base_link.STL"/>
         </geometry>
+        <!-- Origin of the visual element. xyz is in metres. rpy stands for roll pitch yaw in radians. -->
         <origin xyz="0 0 0.025" rpy="1.5707963 0 0"/>
       </visual>
+      <!-- Defines the collision boundaries. -->
       <collision>
+        <!-- Shape of object. -->
         <geometry>
           <mesh filename="package://claw_description/meshes/base_link.STL"/>
         </geometry>
+        <!-- Collision origin is usually the same as the visual origin. -->
         <origin xyz="0 0 0.025" rpy="1.5707963 0 0"/>
       </collision>
+      <!--
+        Defines the inertial properties of the link.
+        If this block is not defined, everything defaults to zero. However, Gazebo will not render the link if inertia values are zero.
+       -->
       <inertial>
         <origin xyz="0 0 0" rpy="0 0 0"/>
@@ -29,9 +56,17 @@
       </inertial>
     </link>
+    <!--
+      Defines a joint between base_link and claw1.
+      Continuous joint rotates about an axis with no bounds. Ideally, this joint should be revolute.
+      To find out the other types of joints: http://wiki.ros.org/urdf/XML/joint#Attributes
+    -->
     <joint name="${prefix}joint1" type="continuous">
+      <!-- Origin of the joint which also defines how the 2 links are relative to each other. -->
       <origin xyz="0.05251 -0.010729 -0.0375" rpy="-1.5708 ${pi} 3.1416"/>
       <parent link="${prefix}base_link"/>
       <child link="${prefix}claw1"/>
+      <!-- Which axis is the continuous joint about. -->
       <axis xyz="0 0 1"/>
+      <!-- Add damping and friction coefficients to this joint. -->
       <dynamics damping="0.1" friction="0.1"/>
     </joint>
@@ -63,5 +98,4 @@
         <origin xyz="0 0 0" rpy="0 0 0"/>
       </collision>
-      <!-- Some inertia values have to be non-zero for this link to render in Gazebo. We set ixx, iyy, izz to 1.0 -->
       <inertial>
         <origin xyz="-0.0185468224648669 0.110151443507784 -0.0107513372089238" rpy="0 0 0"/>
@@ -117,15 +151,20 @@
       </inertial>
     </link>
-    <!-- This block connects the joint to an actuator, which informs both simulation and visualization of the robot -->
+    <!-- Transmission block states that the joint has an actuator. -->
     <transmission name="${prefix}joint1_trans">
       <type>transmission_interface/SimpleTransmission</type>
       <actuator name="${prefix}joint1_motor">
+        <!-- Specify the reduction to mimic gearing. -->
         <mechanicalReduction>1</mechanicalReduction>
       </actuator>
+      <!-- Pick the joint to add an actuator. -->
       <joint name="${prefix}joint1">
+        <!-- Actuator will be controlled by an effort joint controller so require an interface for that. -->
         <hardwareInterface>hardware_interface/EffortJointInterface</hardwareInterface>
       </joint>
     </transmission>
+    <!-- Gazebo tag to specify additional properties for simulation in Gazebo. -->
     <gazebo>
+      <!-- Apply the mimic_joint_plugin onto joint2 mimicing joint1. -->
       <plugin name="${prefix}joint2_mimic_plugin" filename="libroboticsgroup_gazebo_mimic_joint_plugin.so">
         <joint>${prefix}joint1</joint>
@@ -134,4 +173,5 @@
     </gazebo>
     <gazebo>
+      <!-- Apply the mimic_joint_plugin onto joint3 mimicing joint1. -->
       <plugin name="${prefix}joint3_mimic_plugin" filename="libroboticsgroup_gazebo_mimic_joint_plugin.so">
         <joint>${prefix}joint1</joint>

File: claw_example/claw_description/urdf/claw.xacro (robot description, xacro)
@@ -1,9 +1,15 @@
+<!-- The purpose of this file is to fix the claw to some abstract link so the claw can be used in the world. -->
 <?xml version="1.0" ?>
 <robot name="claw" xmlns:xacro="http://ros.org/wiki/xacro">
+  <!-- Including the claw.urdf.xacro file to give scope to xacro:claw. Inclusion is a simple copy-and-paste of code. -->
   <xacro:include filename="$(find claw_description)/urdf/claw.urdf.xacro" />
+  <!-- This is the abstract link which the base of the claw attaches to. -->
   <link name="claw_root_link" />
+  <!-- Instantiate the claw by using its macro. -->
   <xacro:claw prefix="" parent="claw_root_link" >
+    <!-- Note that we are passing in a tag as an argument. -->
     <origin xyz="0 0 0" rpy="0 0 0"/>
   </xacro:claw>
+  <!-- This plugin allows the claw to be controlled in gazebo (not important until later). -->
   <gazebo>
     <plugin name="gazebo_ros_control" filename="libgazebo_ros_control.so">
